Commit message: finished?

File: urdf/simple_robot.urdf (robot description, URDF)
Before this commit: robot pi_robot, 12 links, 11 joints
Links:
- removed link base_link
- removed link gripper_base
- removed link jointlink_1
- removed link jointlink_2
- removed link jointlink_3
- removed link left_fingertip
- removed link link_1
- removed link link_2
- removed link link_3
- removed link right_fingertip
- removed link torso_link
- removed link upper_base_link
- added link link0; visual cylinder length=0.05 radius=0.1
- added link link1; visual cylinder length=0.2 radius=0.05
- added link link10, mass 1; collision box size=0.025 .05 0.025; visual box size=0.025 .05 0.025
- added link link2; visual sphere radius=0.052
- added link link3; visual cylinder length=0.2 radius=0.05
- added link link4; visual sphere radius=0.052
- added link link5; visual cylinder length=0.2 radius=0.05
- added link link6; visual sphere radius=0.052
- added link link7; visual cylinder length=0.2 radius=0.05
- added link link8, mass 1; collision box size=0.105 .02 .025; visual box size=0.105 .02 .025
- added link link9, mass 1; collision box size=0.025 .05 0.025; visual box size=0.025 .05 0.025
Joints:
- removed joint base_joint
- removed joint gripper_base_to_left_fingertip
- removed joint gripper_base_to_right_fingertip
- removed joint gripper_joint
- removed joint joint_1
- removed joint joint_2
- removed joint joint_3
- removed joint jointlink_1_link_1
- removed joint jointlink_2_link_2
- removed joint jointlink_3_link_3
- removed joint torso_joint
- added joint joint0: type revolute, parent link0, child link1, origin xyz=0 0 0.10 rpy=0 0 0, axis 0 0 1, limit lower=-0.6 upper=0.6 effort=0 velocity=3
- added joint joint1: type revolute, parent link1, child link2, origin xyz=0 0 0.1 rpy=0 0 0, axis 0 1 0, limit lower=0 upper=1.6 effort=10 velocity=3
- added joint joint2: type fixed, parent link2, child link3, origin xyz=0 0 0.1 rpy=0 0 0, axis 0 0 1
- added joint joint3: type revolute, parent link3, child link4, origin xyz=0 0 0.1 rpy=0 0 0, axis 0 1 0, limit lower=-1.57 upper=1.57 effort=10 velocity=3
- added joint joint4: type fixed, parent link4, child link5, origin xyz=0 0 0.1 rpy=0 0 0, axis 0 0 1
- added joint joint5: type revolute, parent link5, child link6, origin xyz=0 0 0.1 rpy=0 0 0, axis 0 1 0, limit lower=-1.57 upper=1.57 effort=10 velocity=3
- added joint joint6: type fixed, parent link6, child link7, origin xyz=0 0 0.1 rpy=0 0 0, axis 0 0 1
- added joint joint7: type revolute, parent link7, child link8, origin xyz=0 0 0 rpy=-1.5708 0  0, axis 0 1 0, limit lower=-1.57 upper=1.57 effort=10 velocity=3
- added joint joint8: type prismatic, parent link8, child link9, origin xyz=0.04 -0.135 -0.0, axis 1 0 0, limit lower=-0.03 upper=0.0 effort=1.0 velocity=0.5
- added joint joint9: type prismatic, parent link8, child link10, origin xyz=-0.04 -0.135 0.0, axis 1 0 0, limit lower=0 upper=0.03 effort=1.0 velocity=0.5
